Commit message: ORB SLAM
Pridavanie ORB SLAMu na simulaciu s hlbkovym senzorom ktora uz fungovala.

File: src/m2wr_description/urdf/m2wr.xacro (robot description, xacro)
@@ -40,5 +40,5 @@
     <material>Gazebo/Blue</material>
   </gazebo>
- <gazebo reference="sensor_laser">
+ <gazebo reference="camera_link">
     <material>Gazebo/Red</material>
   </gazebo>
@@ -48,6 +48,6 @@
       <alwaysOn>true</alwaysOn>
       <updateRate>20</updateRate>
-      <leftJoint>joint_right_wheel</leftJoint> !!mam to naopak!!
-      <rightJoint>joint_left_wheel</rightJoint>
+      <leftJoint>joint_left_wheel</leftJoint> <!-- Toto bolo naopak -->
+      <rightJoint>joint_right_wheel</rightJoint>
       <frontJoint>joint_front_wheel</frontJoint>
       <backJoint>joint_back_wheel</backJoint>
@@ -61,33 +61,52 @@
     </plugin>
   </gazebo>
-  <gazebo reference="sensor_laser">
-    <sensor type="ray" name="head_hokuyo_sensor">
-      <pose>0 0 0 0 0 0</pose>
+  <gazebo reference="camera_link">
+    <sensor type="depth" name="kinect_sensor">
+      <pose frame="camera_link">0 0 0 0 1.5707 0</pose>
       <visualize>true</visualize>
       <update_rate>100</update_rate>
-      <ray>
-        <scan>
-          <horizontal>
-            <samples>666</samples>
-            <resolution>1</resolution>
-            <min_angle>-2.0943951024</min_angle>
-            <max_angle>2.0943951024</max_angle>
-          </horizontal>
-        </scan>
-        <range>
-          <min>0.10</min>
-          <max>5.6</max>
-          <resolution>0.01</resolution>
-        </range>
-        <noise>
-          <type>gaussian</type>
-          <mean>0.0</mean>
-          <stddev>0.01</stddev>
-        </noise>
-      </ray>
-      <plugin name="gazebo_ros_head_hokuyo_controller" filename="libgazebo_ros_laser.so">
-        <topicName>/m2wr/laser/scan</topicName>
-        <frameName>sensor_laser</frameName>
-      </plugin>
+      <camera>
+          <horizontal_fov>1.047198</horizontal_fov>
+          <image>
+            <width>1024</width>
+            <height>1024</height>
+            <format>R8G8B8</format>
+          </image>
+          <clip>
+            <near>0.25</near>
+            <far>5.46</far>
+          </clip>
+          <noise>
+              <type>gaussian</type>
+              <mean>0.5</mean>
+              <stddev>1.0</stddev>
+          </noise>
+        </camera>
+      <plugin name="camera_plugin" filename="libgazebo_ros_openni_kinect.so">
+          <baseline>0.2</baseline>
+          <alwaysOn>true</alwaysOn>
+          <!-- Keep this zero, update_rate in the parent <sensor> tag
+            will control the frame rate. -->
+          <updateRate>0.0</updateRate>
+          <cameraName>kinect_sensor</cameraName>
+          <imageTopicName>/camera/rgb/image_raw</imageTopicName>
+          <cameraInfoTopicName>/camera/rgb/camera_info</cameraInfoTopicName>
+          <depthImageTopicName>/camera/depth_registered/image_raw</depthImageTopicName>
+          <depthImageCameraInfoTopicName>/camera/depth_registered/camera_info</depthImageCameraInfoTopicName>
+          <pointCloudTopicName>/camera/depth_registered/points</pointCloudTopicName>
+          <frameName>camera_link_optical</frameName>
+          <pointCloudCutoff>0.5</pointCloudCutoff>
+          <pointCloudCutoffMax>3.0</pointCloudCutoffMax>
+          <distortionK1>0</distortionK1>
+          <distortionK2>0</distortionK2>
+          <distortionK3>0</distortionK3>
+          <distortionT1>0</distortionT1>
+          <distortionT2>0</distortionT2>
+          <CxPrime>0</CxPrime>
+          <Cx>0</Cx>
+          <Cy>0</Cy>
+          <focalLength>0</focalLength>
+          <hackBaseline>0</hackBaseline>
+        </plugin>
     </sensor>
   </gazebo>
@@ -129,5 +148,5 @@
     </visual>
   </link>
-  <link name="sensor_laser">
+  <link name="camera_link">
     <inertial>
 	<mass value="0.1" />
@@ -149,9 +168,25 @@
     </collision>
     </link>
-    <joint name="joint_sensor_laser" type="fixed">
-    <origin xyz="0.43 0.43 -0.22" rpy="0 0 0.53"/>
-    <parent link="link_chassis"/>
-    <child link="sensor_laser"/>
-  </joint>
+    <joint name="joint_camera" type="fixed">
+    <origin xyz="0.23 -0.06 -0.11" rpy="0 0 0"/>
+    <parent link="link_chassis"/>
+    <child link="camera_link"/>
+  </joint>
+  <joint name="camera_optical_joint" type="fixed">
+    <!-- these values have to be these values otherwise the gazebo camera
+        image won't be aligned properly with the frame it is supposedly
+        originating from -->
+    <origin xyz="0 0 0" rpy="-1.5708 0 -1.5708"/>
+    <parent link="camera_link"/>
+    <child link="camera_link_optical"/>
+  </joint>
+  <link name="camera_link_optical">
+  </link>
+  <joint name="camera_link_joint" type="fixed">
+        <origin xyz="0 0 0.6"
+                rpy="0 0 0" />
+        <parent link="link_chassis"/>
+        <child link="camera_link"/>
+    </joint>
   <link name="link_right_wheel">
     <inertial>

Commit message: Pridavanie RTABmapu
Pridal som RTABmap aj este niektore casti

V rtabmap launch subore som zmenil len nech sa rviz spusta namiest rtabmapvizu

File: src/m2wr_description/urdf/m2wr.xacro (robot description, xacro)
@@ -169,5 +169,5 @@
     </link>
     <joint name="joint_camera" type="fixed">
-    <origin xyz="0.23 -0.06 -0.11" rpy="0 0 0"/>
+    <origin xyz="0.23 -0.06 0.11" rpy="0 0 0"/>
     <parent link="link_chassis"/>
     <child link="camera_link"/>

Commit message: RTABMap a ORB-SLAM
RTABMap a ORB-SLAM maju rovnake parametre pre launch subory.

File: src/m2wr_description/urdf/m2wr.xacro (robot description, xacro)
@@ -25,5 +25,5 @@
     <color rgba="1.0 1.0 1.0 1.0"/>
   </material>
-  <gazebo reference="link_chassis">
+  <gazebo reference="base_link">
     <material>Gazebo/White</material>
   </gazebo>
@@ -58,5 +58,5 @@
       <odometryTopic>odom</odometryTopic>
       <odometryFrame>odom</odometryFrame>
-      <robotBaseFrame>link_chassis</robotBaseFrame>
+      <robotBaseFrame>base_link</robotBaseFrame>
     </plugin>
   </gazebo>
@@ -111,5 +111,5 @@
     </sensor>
   </gazebo>
-  <link name="link_chassis">
+  <link name="base_link">
     <!-- pose and inertial -->
     <pose>0 0 0.1 0 0 0</pose>
@@ -170,5 +170,5 @@
     <joint name="joint_camera" type="fixed">
     <origin xyz="0.23 -0.06 0.11" rpy="0 0 0"/>
-    <parent link="link_chassis"/>
+    <parent link="base_link"/>
     <child link="camera_link"/>
   </joint>
@@ -186,5 +186,5 @@
         <origin xyz="0 0 0.6"
                 rpy="0 0 0" />
-        <parent link="link_chassis"/>
+        <parent link="base_link"/>
         <child link="camera_link"/>
     </joint>
@@ -211,5 +211,5 @@
     <origin rpy="0 0 0" xyz="0 0.30 -0.23"/>
     <child link="link_right_wheel"/>
-    <parent link="link_chassis"/>
+    <parent link="base_link"/>
     <axis rpy="0 0 0" xyz="0 1 0"/>
     <limit effort="10000" velocity="1000"/>
@@ -238,5 +238,5 @@
     <origin rpy="0 0 0" xyz="0 -0.30 -0.23"/>
     <child link="link_left_wheel"/>
-    <parent link="link_chassis"/>
+    <parent link="base_link"/>
     <axis rpy="0 0 0" xyz="0 1 0"/>
     <limit effort="10000" velocity="1000"/>
@@ -265,5 +265,5 @@
     <origin rpy="0 0 0" xyz="0.3 0 -0.28"/>
     <child link="link_front_wheel"/>
-    <parent link="link_chassis"/>
+    <parent link="base_link"/>
     <axis rpy="0 0 0" xyz="0 1 0"/>
     <limit effort="10000" velocity="1000"/>
@@ -292,5 +292,5 @@
     <origin rpy="0 0 0" xyz="-0.35 0 -0.28"/>
     <child link="link_back_wheel"/>
-    <parent link="link_chassis"/>
+    <parent link="base_link"/>
     <axis rpy="0 0 0" xyz="0 1 0"/>
     <limit effort="10000" velocity="1000"/>
